File: power2.kicad_pcb (KiCad board)
At the start: 2 copper layers, 99.7 x 100.3 mm, 212 parts, among them J1 USB_A, J2 Barrel_Jack_Switch, J3 Conn_02x06_Odd_Even, J4 Conn_02x10_Odd_Even, J5 Conn_02x06, J6 Conn_02x10_Odd_Even, J7 Conn_Coaxial, J8 Conn_Coaxial, Q1 MOSFET_P, T1 BALUN, T2 BALUN, U1 ZLDO1117G33TA, U10 lx9_XC6SLX9-TQ144, U11 FSM1LPTR, U12 FSM1LPTR, U13 FSM1LPTR, U14 SI5351C, U15 MAX5864, U16 MAX2830, U2 ZLDO1117G33TA, U3 ZLDO1117G33TA, U4 FSM1LPTR, U5 STM32F722ZET, U6 LSM9DS1, U7 Omega2+, U8 FSM1LPTR, U9 CY7C199, X1 Oscillator_ASE-xxxMHz, Y1 ABM8G-16.000MHZ-B4Y-T, Y2 Crystal, Y3 ABM8G-25.000MHZ-B4Y-T

Commit message: diseño de esquematico CASI FINAL
Parts:
- moved R20 15.3 mm to (123.2, 95.2), turned to 90 degrees
- moved C35 7.21 mm to (108.7, 90.0), turned to 180 degrees
- moved R12 5.66 mm to (108.0, 29.1)
- moved R14 5.66 mm to (108.0, 25.0)
- moved R15 5.66 mm to (108.0, 23.0)
- moved R13 5.66 mm to (108.0, 26.9)
- moved J5 4.76 mm to (134.6, 17.9)
- moved U7 2.68 mm to (104.0, 47.0)
- moved R30 0.66 mm to (88.8, 86.1), turned to 270 degrees
- moved C44 0.64 mm to (76.4, 47.3)
- moved C45 0.64 mm to (73.7, 47.3)
Connections:
- J3 pad 10: /STM32_micro/SDO_A_G -> /STM32_micro/CS_A_G
- J3 pad 3: /STM32_micro/INT1_A_G -> /STM32_micro/INT_M
- J3 pad 5: /STM32_micro/INT_M -> /STM32_micro/DRDY_M
- J3 pad 6: /STM32_micro/DRDY_M -> /STM32_micro/INT1_A_G
- J3 pad 7: /STM32_micro/CS_M -> /STM32_micro/SDO_M
- J3 pad 8: /STM32_micro/CS_A_G -> /STM32_micro/SDO_A_G
- J3 pad 9: /STM32_micro/SDO_M -> /STM32_micro/CS_M
- J5 pad 10: /ONION_OMEGA/SPI_CS -> /ONION_OMEGA/MOSI
- J5 pad 11: VCC_5V -> /ONION_OMEGA/MISO
- J5 pad 2: GND -> I2C_SCL
- J5 pad 4: /ONION_OMEGA/MISO -> /ONION_OMEGA/RX_PIN
- J5 pad 5: I2C_SCL -> /ONION_OMEGA/TX_PIN
- J5 pad 6: /ONION_OMEGA/MOSI -> VCC_5V
- J5 pad 7: /ONION_OMEGA/RX_PIN -> GND
- J5 pad 8: /ONION_OMEGA/SPI_CLK -> /ONION_OMEGA/SPI_CS
- J5 pad 9: /ONION_OMEGA/TX_PIN -> /ONION_OMEGA/SPI_CLK
Routing:
- net I2C_SDA: track 214.3 -> 70.1 mm, vias 6 -> 3
- net I2C_SCL: track 194.8 -> 59.4 mm, vias 4 -> 1
- net /FPGA_spartan6/FSW_1: track 100.3 -> 0.00 mm, vias 6 -> 0
- net JNRST: track 122.6 -> 39.7 mm, vias 5 -> 4
- net USART_TX: track 75.2 -> 0.00 mm, vias 1 -> 0
- net USART_RX: track 75.2 -> 0.00 mm, vias 1 -> 0
- net JTDO_OMEGA: track 69.2 -> 0.00 mm, vias 6 -> 0
- net BOOT0: track 67.7 -> 0.00 mm, vias 4 -> 0
- net /ONION_OMEGA/RX_PIN: track 53.4 -> 0.00 mm, vias 1 -> 0
- net /ONION_OMEGA/TX_PIN: track 50.1 -> 0.00 mm
- net JTMS: track 76.9 -> 26.8 mm, vias 4 -> 1
- net JTDO: track 48.4 -> 0.00 mm, vias 1 -> 0
- net /FPGA_spartan6/DONE: track 48.4 -> 0.00 mm, vias 1 -> 0
- net JTCK: track 76.3 -> 29.1 mm, vias 4 -> 1
- net JTRST: track 42.6 -> 0.00 mm, vias 3 -> 0
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