File: FPGA_spartan6.sch (KiCad schematic (older format))
At the start: 81 parts

Commit message: asignacion pines de control
Parts:
- added D? (x5): LED, LED_SMD:LED_0603_1608Metric, symbol BAT2032:LED
- added R? (x2): 220, Resistor_SMD:R_0603_1608Metric_Pad1.05x0.95mm_HandSolder, symbol BAT2032:R
- added R?: 4.7k, Resistor_SMD:R_0603_1608Metric_Pad1.05x0.95mm_HandSolder, symbol BAT2032:R
- added R? (x4): 600, Resistor_SMD:R_0603_1608Metric_Pad1.05x0.95mm_HandSolder, symbol BAT2032:R
- added U?: FSM1LPTR, SWITCH_FSM1LPA, symbol FSM1LPTR:FSM1LPTR
- U?: footprint (none) -> Package_SO:TSOP-I-28_11.8x8mm_P0.55mm; Digikey (none) -> 428-2013-ND
Connections:
- net labels added: DONE, FMC_A0, FMC_A1, FMC_A2, FMC_A3, FMC_A4, FMC_A5, FMC_A6, FMC_A7, FMC_A[7...0], FMC_D0, FMC_D1, FMC_D10, FMC_D11, FMC_D12, FMC_D13, FMC_D14, FMC_D15, FMC_D2, FMC_D3, FMC_D4, FMC_D5, FMC_D6, FMC_D7, FMC_D8, FMC_D9, FMC_D[15...0], FMC_N_DOUT, FPGA_TDI, FPGA_TDO, JTCK, JTDI_FPGA, JTDO_OMEGA, JTMS, PROGRAM_B, TCK, TMS
- wire segments 317 -> 399
- no-connect marks 0 -> 1
Other:
- moved on the sheet: R?

Commit message: asignacion pines de control
Parts:
- removed J? (x2): Conn_02x06, Connector_PinHeader_2.54mm:PinHeader_2x06_P2.54mm_Vertical, symbol Connector_Generic:Conn_02x06_Counter_Clockwise
- removed R? (x4): 10k, Resistor_SMD:R_0603_1608Metric_Pad1.05x0.95mm_HandSolder, symbol BAT2032:R
- removed R? (x16): 200, Resistor_SMD:R_0603_1608Metric_Pad1.05x0.95mm_HandSolder, symbol BAT2032:R
- removed U? (x2): FSM1LPTR, SWITCH_FSM1LPA, symbol FSM1LPTR:FSM1LPTR
- U10: renamed from U?; footprint (none) -> Package_QFP:LQFP-144_20x20mm_P0.5mm; digiker (none) -> 122-1745-ND
- X1: renamed from X?; footprint Oscillator:Oscillator_SMD_Abracon_ASE-4Pin_3.2x2.5mm -> Oscillator:Oscillator_SMD_Abracon_ASE-4Pin_3.2x2.5mm_HandSoldering; digikey 576-5011-5-ND -> 535-11114-1-ND
- gave numbers to parts that had none: 68
Connections:
- net labels added: adDA0, adDA1, adDA2, adDA3, adDA4, adDA5, adDA6, adDA7, adDD0, adDD1, adDD2, adDD3, adDD4, adDD5, adDD6, adDD7, adDD8, adDD9
- net labels removed: FGPIO16, FGPIO17, FGPIO18, FGPIO19, FGPIO20, FGPIO21, FGPIO22, FGPIO23, FGPIO24, FGPIO25, FGPIO26, FGPIO27, FGPIO28, FGPIO29, FGPIO30, FGPIO31, FSW_3, FSW_4
- wire segments 399 -> 356
- no-connect marks 1 -> 7

Commit message: retoque casi finales
Parts:
- removed J5: Conn_02x06_Odd_Even, Connector_PinHeader_2.54mm:PinHeader_2x06_P2.54mm_Vertical, symbol Connector_Generic:Conn_02x06_Odd_Even
- removed J6: Conn_02x06, Connector_PinHeader_2.54mm:PinHeader_2x06_P2.54mm_Vertical, symbol Connector_Generic:Conn_02x06_Counter_Clockwise
- removed R15, R16, R17, R18, R19, R20, R21, R22, R23, R24, R25, R26, R27, R28, R29, R30: 200, Resistor_SMD:R_0603_1608Metric_Pad1.05x0.95mm_HandSolder, symbol BAT2032:R
- added J6: Conn_02x10_Odd_Even, Connector_PinHeader_2.54mm:PinHeader_2x10_P2.54mm_Vertical, symbol Connector_Generic:Conn_02x10_Odd_Even
- C45: value 1uF -> 0.1uF
- C51: value 4.7uF -> 0.1uF
- D10, D6, D7, D8, D9: footprint LED_SMD:LED_0603_1608Metric -> LED_SMD:LED_0603_1608Metric_Pad1.05x0.95mm_HandSolder
- U10: symbol pcb_edu-cache:lx9_XC6SLX9-TQ144 -> power-rescue:lx9_XC6SLX9-TQ144-pcb_edu-cache
- X1: symbol pcb_edu-cache:Oscillator_ASE-xxxMHz -> power-rescue:Oscillator_ASE-xxxMHz-pcb_edu-cache
Connections:
- net labels added: +5V, FMC_A[0..7], FMC_D[0..15], FMC_NE1, FMC_NWAIT, FMC_[0..7], GCK0, GCK1, I2C_0[0..1], JTAG0, JTAG1, JTAG2, JTAG3, JTAG4, JTAG5, JTAG[0..5], NRST, TDI, TDO, TRST
- net labels removed: FMC_A[7...0], FMC_CONTROL, FMC_D[15...0], I2C_0[1..0]
- wire segments 356 -> 351
- no-connect marks 7 -> 3

Commit message: diseño de esquematico
Parts:
- removed C45, C53: 0.1uF, Capacitor_SMD:C_0603_1608Metric_Pad1.05x0.95mm_HandSolder, symbol Device:C
- removed C46, C49, C52, C59, C72, C73: 4.7uF, Capacitor_SMD:C_0603_1608Metric_Pad1.05x0.95mm_HandSolder, symbol Device:C
- removed D8, D9: LED, LED_SMD:LED_0603_1608Metric_Pad1.05x0.95mm_HandSolder, symbol BAT2032:LED
- removed R33, R34: 600, Resistor_SMD:R_0603_1608Metric_Pad1.05x0.95mm_HandSolder, symbol BAT2032:R
- added C58, C63, C66, C82: 4.7uF, Capacitor_SMD:C_0603_1608Metric_Pad1.05x0.95mm_HandSolder, symbol Device:C
- added C70: 0.47uF, Capacitor_SMD:C_0603_1608Metric_Pad1.05x0.95mm_HandSolder, symbol Device:C
- C47, C48, C54, C60: value 0.1uF -> 4.7uF
- C49: renamed from C58; value 0.1uF -> 4.7uF
- C50, C51, C56: value 0.1uF -> 0.47uF
- C53: renamed from C61; value 0.1uF -> 4.7uF
- C55, C62, C67, C68, C69, C71: value 4.7uF -> 0.47uF
- C57: renamed from C63; value 0.1uF -> 4.7uF
- C59: renamed from C66; value 0.1uF -> 4.7uF
- C61: renamed from C70; value 0.1uF -> 4.7uF
- U11, U12, U13: footprint SWITCH_FSM1LPA -> library:FSM1LPTR
- renumbered C57 to C52, C74 to C72, D7 to D10, D10 to D11, D6 to D9, R31 to R18, R32 to R19, R35 to R20, R36 to R21, R37 to R22, R38 to R23, R39 to R24, R40 to R25, R41 to R26
Connections:
- net labels added: FPGA_JTDO
- net labels removed: FMC_A[0..7], FMC_D[0..15], FMC_[0..7], I2C_00, I2C_01, I2C_0[0..1], JTAG0, JTAG1, JTAG2, JTAG3, JTAG4, JTAG5, JTAG[0..5], JTDI_FPGA, NRST, TDI, TDO, TRST
- wire segments 351 -> 342
- no-connect marks 3 -> 4
Other:
- note added: "VCCAUX"
- note added: "VCCINT"
- note added: "VCCO_0"
- note added: "VCCO_1"
- note added: "VCCO_2"
- note added: "VCCO_3\n"
- moved on the sheet: C49, C52, C53, C57, C59, C61, J6, U9
